File: ESP-32_WLED-Controller_Addon/KiCad7_Project/ESP-32_WLED-Controller_Addon.kicad_sch (KiCad schematic)
At the start: 11 parts, among them J1 Conn_01x05_Female, J2 Conn_01x02_Female, J3 AudioJack4, J4 Conn_01x02_Female, J5 Conn_01x04_Female

Commit message: fixed small issues in BOM
Parts:
- C1, C2: now in the parts list
- J1, J2, J4, J5: now left out of the parts list
Changed lines of the file:
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@@
   )
   (symbol (lib_id "Connector:Conn_01x02_Female") (at 129.54 138.43 0) (unit 1)
-    (in_bom yes) (on_board yes) (dnp no) (fields_autoplaced)
+    (in_bom no) (on_board yes) (dnp no) (fields_autoplaced)
     (property "Reference" "J2" (at 131.445 138.4299 0)
       (effects (font (size 1.27 1.27)) (justify left))
@@
   )
   (symbol (lib_id "Connector:Conn_01x02_Female") (at 130.175 118.745 0) (unit 1)
-    (in_bom yes) (on_board yes) (dnp no) (fields_autoplaced)
+    (in_bom no) (on_board yes) (dnp no) (fields_autoplaced)
     (property "Reference" "J4" (at 132.08 118.7449 0)
       (effects (font (size 1.27 1.27)) (justify left))
@@
   )
   (symbol (lib_id "Connector:Conn_01x04_Female") (at 49.53 105.41 0) (unit 1)
-    (in_bom yes) (on_board yes) (dnp no) (fields_autoplaced)
+    (in_bom no) (on_board yes) (dnp no) (fields_autoplaced)
     (property "Reference" "J5" (at 50.8 105.4099 0)
       (effects (font (size 1.27 1.27)) (justify left))
@@
   )
   (symbol (lib_id "Device:C") (at 217.805 74.295 270) (unit 1)
-    (in_bom no) (on_board yes) (dnp no)
+    (in_bom yes) (on_board yes) (dnp no)
     (property "Reference" "C2" (at 217.805 81.0514 90)
       (effects (font (size 1.27 1.27)))
@@
   )
   (symbol (lib_id "Connector:Conn_01x05_Female") (at 44.45 71.755 0) (mirror y) (unit 1)
-    (in_bom yes) (on_board yes) (dnp no) (fields_autoplaced)
+    (in_bom no) (on_board yes) (dnp no) (fields_autoplaced)
     (property "Reference" "J1" (at 45.085 61.595 0)
       (effects (font (size 1.27 1.27)))
@@
   )
   (symbol (lib_id "Device:C") (at 217.805 67.945 90) (unit 1)
-    (in_bom no) (on_board yes) (dnp no)
+    (in_bom yes) (on_board yes) (dnp no)
     (property "Reference" "C1" (at 217.805 61.1886 90)
       (effects (font (size 1.27 1.27)))
